File: Main/Main.kicad_pcb (KiCad board)
At the start: 2 copper layers, 90 x 100 mm, 49 parts, among them J1 Battery_Conn, J10 SWD_Conn, J2 Display_Conn, J3 Keypad_Conn, J4 Mux_Conn, J5 USB_B_Micro, M1 Motor_DC, Q1 IRLML5203, Q2 MMBT5550L, Q3 MMBT5550L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

Commit message: Continued progress
Parts:
- moved C17 169.3 mm to (194.3, 54.6)
- moved C23 168.3 mm to (200.7, 82.5), turned to 270 degrees
- moved U6 166.5 mm to (201.9, 54.6)
- moved D6 142.6 mm to (194.3, 66.0), turned to 180 degrees
- moved R20 134.8 mm to (198.1, 72.4), turned to 90 degrees
- moved U8 132.3 mm to (193.0, 72.4), turned to 180 degrees
- moved C22 122.2 mm to (204.5, 97.8), turned to 90 degrees
- moved C21 120.0 mm to (199.4, 97.8), turned to 90 degrees
- moved C20 117.0 mm to (194.3, 97.8), turned to 90 degrees
- moved C24 110.1 mm to (190.5, 97.8), turned to 90 degrees
- moved R21 98.4 mm to (198.1, 67.3), turned to 270 degrees
- moved J3 94.3 mm to (221.0, 115.6)
- moved J4 86.5 mm to (276.9, 78.7)
- moved R1 85.2 mm to (220.5, 111.3)
- moved R2 85.2 mm to (223.0, 111.3)
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Connections:
- C1 pad 1: VDD -> +3V3
- C16 pad 1: VDD -> +3V3
- U2 pad 7: VDD -> +3V3
