File: Main/Main.sch (KiCad schematic (older format))
At the start: 49 parts, among them J1 Battery_Conn, J10 SWD_Conn, J11 USB_B_Micro, J2 Display_Conn, J3 Keypad_Conn, J4 Mux_Conn, M1 Motor_DC, Q1 IRLML5203, Q2 MMBT5550L, Q3 MMBT5550L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

Commit message: Check Main for PCB updates
Parts:
- removed J11: USB_B_Micro, digikey-footprints:USB_Micro_B_Female_Vert_1051330001, symbol sink_or_be_sunk-rescue:USB_B_Micro-Connector
- added J5: USB_B_Micro, digikey-footprints:USB_Micro_B_Female_Vert_1051330001, symbol Main:USB_B_Micro
- C23, C24, C25: footprint Capacitor_SMD:C_0805_2012Metric_Pad1.18x1.45mm_HandSolder -> Capacitor_SMD:C_0805_2012Metric_Pad1.15x1.40mm_HandSolder
- U3: footprint PCB_ESP32:SN74HC151N-PDIP -> Main:SN74HC151N-PDIP
Connections:
- wire segments 186 -> 184
Changed lines of the file:
@@
 encoding utf-8
 Sheet 1 1
-Title "Main Layout"
-Date "2021-09-01"
-Rev "1"
-Comp "Sink or be Sunk"
+Title ""
+Date ""
+Rev ""
+Comp ""
 Comment1 ""
 Comment2 ""
@@
 	-1   0    0    -1
 $EndComp
-$Comp
-L sink_or_be_sunk-rescue:USB_B_Micro-Connector J11
-U 1 1 61591780
-P 9750 1250
-F 0 "J11" H 9807 1717 50  0000 C CNN
-F 1 "USB_B_Micro" H 9807 1626 50  0000 C CNN
-F 2 "digikey-footprints:USB_Micro_B_Female_Vert_1051330001" H 9900 1200 50  0001 C CNN
-F 3 "~" H 9900 1200 50  0001 C CNN
-	1    9750 1250
-	-1   0    0    -1
-$EndComp
 NoConn ~ 9250 1450
 $Comp
@@
 Wire Wire Line
 	9000 1800 9000 1750
-Wire Wire Line
-	9850 1650 9850 1750
-Wire Wire Line
-	9850 1750 9750 1750
 Connection ~ 9000 1750
 Wire Wire Line
@@
 Wire Wire Line
 	9750 1650 9750 1750
-Connection ~ 9750 1750
 Wire Wire Line
 	9750 1750 9000 1750
@@
 F 0 "U3" H 2000 5885 50  0000 C CNN
 F 1 "SN74HC151N" H 2000 5976 50  0000 C CNN
-F 2 "PCB_ESP32:SN74HC151N-PDIP" H 2050 6450 50  0001 C CNN
+F 2 "Main:SN74HC151N-PDIP" H 2050 6450 50  0001 C CNN
 F 3 "" H 2050 6450 50  0001 C CNN
 	1    2000 6450
@@
 F 0 "C24" H 6415 6496 50  0000 L CNN
 F 1 "4.7uF" H 6415 6405 50  0000 L CNN
-F 2 "Capacitor_SMD:C_0805_2012Metric_Pad1.18x1.45mm_HandSolder" H 6338 6300 50  0001 C CNN
+F 2 "Capacitor_SMD:C_0805_2012Metric_Pad1.15x1.40mm_HandSolder" H 6338 6300 50  0001 C CNN
 F 3 "~" H 6300 6450 50  0001 C CNN
 	1    6300 6450
@@
 F 0 "C23" H 5865 6496 50  0000 L CNN
 F 1 "4.7uF" H 5865 6405 50  0000 L CNN
-F 2 "Capacitor_SMD:C_0805_2012Metric_Pad1.18x1.45mm_HandSolder" H 5788 6300 50  0001 C CNN
+F 2 "Capacitor_SMD:C_0805_2012Metric_Pad1.15x1.40mm_HandSolder" H 5788 6300 50  0001 C CNN
 F 3 "~" H 5750 6450 50  0001 C CNN
 	1    5750 6450
@@
 F 0 "C25" H 10865 4596 50  0000 L CNN
 F 1 "1uF" H 10865 4505 50  0000 L CNN
-F 2 "Capacitor_SMD:C_0805_2012Metric_Pad1.18x1.45mm_HandSolder" H 10788 4400 50  0001 C CNN
+F 2 "Capacitor_SMD:C_0805_2012Metric_Pad1.15x1.40mm_HandSolder" H 10788 4400 50  0001 C CNN
 F 3 "~" H 10750 4550 50  0001 C CNN
 	1    10750 4550
@@
 	-1   0    0    -1
 $EndComp
+$Comp
+L Main:USB_B_Micro J5
+U 1 1 6163041A
+P 9750 1250
+F 0 "J5" H 9520 1239 50  0000 R CNN
+F 1 "USB_B_Micro" H 9520 1148 50  0000 R CNN
+F 2 "digikey-footprints:USB_Micro_B_Female_Vert_1051330001" H 9900 1200 50  0001 C CNN
+F 3 "~" H 9900 1200 50  0001 C CNN
+	1    9750 1250
+	-1   0    0    -1
+$EndComp

Commit message: Continued progress
Connections:
- net VDD is gone; now on net +3V3: C1.1, C16.1, U2.7
Changed lines of the file:
@@
 Wire Wire Line
 	4400 4950 4500 4950
-$Comp
-L power:VDD #PWR?
-U 1 1 615C22A9
-P 4500 4400
-AR Path="/6144DCFC/615C22A9" Ref="#PWR?"  Part="1"
-AR Path="/615C22A9" Ref="#PWR08"  Part="1"
-F 0 "#PWR08" H 4500 4250 50  0001 C CNN
-F 1 "VDD" H 4515 4573 50  0000 C CNN
-F 2 "" H 4500 4400 50  0001 C CNN
-F 3 "" H 4500 4400 50  0001 C CNN
-	1    4500 4400
-	1    0    0    -1
-$EndComp
 Wire Wire Line
 	4200 4700 4150 4700
@@
 F 3 "~" H 7650 6100 50  0001 C CNN
 	1    7650 6100
-	1    0    0    -1
-$EndComp
-$Comp
-L power:VDD #PWR06
-U 1 1 616B30A6
-P 7400 5950
-F 0 "#PWR06" H 7400 5800 50  0001 C CNN
-F 1 "VDD" H 7417 6123 50  0000 C CNN
-F 2 "" H 7400 5950 50  0001 C CNN
-F 3 "" H 7400 5950 50  0001 C CNN
-	1    7400 5950
 	1    0    0    -1
 $EndComp
@@
 Wire Notes Line
 	550  7150 550  5650
-Wire Wire Line
-	7150 5950 7400 5950
-Connection ~ 7400 5950
-Wire Wire Line
-	7400 5950 7650 5950
 $Comp
 L Battery_Management:MCP73831-2-OT U8
@@
 	-1   0    0    -1
 $EndComp
+$Comp
+L power:+3.3V #PWR0112
+U 1 1 61600BF1
+P 4500 4400
+F 0 "#PWR0112" H 4500 4250 50  0001 C CNN
+F 1 "+3.3V" H 4515 4573 50  0000 C CNN
+F 2 "" H 4500 4400 50  0001 C CNN
+F 3 "" H 4500 4400 50  0001 C CNN
+	1    4500 4400
+	1    0    0    -1
+$EndComp
+Wire Wire Line
+	7150 5950 7400 5950
+$Comp
+L power:+3.3V #PWR0113
+U 1 1 61604395
+P 7400 5950
+F 0 "#PWR0113" H 7400 5800 50  0001 C CNN
+F 1 "+3.3V" H 7415 6123 50  0000 C CNN
+F 2 "" H 7400 5950 50  0001 C CNN
+F 3 "" H 7400 5950 50  0001 C CNN
+	1    7400 5950
+	1    0    0    -1
+$EndComp
+Connection ~ 7400 5950
+Wire Wire Line
+	7400 5950 7650 5950
 $EndSCHEMATC
