File: sink_or_be_sunk.kicad_pcb (KiCad board)
At the start: 2 copper layers, 86.1 x 82.3 mm, 81 parts, among them J1 Grid_Conn, J10 640456-2, J11 640456-2, J12 640456-2, J13 640456-2, J14 640456-2, J15 640456-2, J16 640456-2, J17 USB_B_Micro, J18 Keypad_Conn, J19 Display_Conn, J2 640456-6, J20 JTAG_Conn, J21 Debug_Conn, J22 Battery_Conn, J3 640456-6, J4 640456-6, J5 640456-6, J6 640456-6, J7 640456-6, J8 640456-6, J9 640456-2, M1 Motor_DC, Q1 IRL530, Q2 Q_PMOS_GDS, Q3 2N3704, Q4 2N3704, SW1 SW_DPST, SW2 Reset_SW, U1 SN74HC151N, U3 MCP73831-2-OT, U4 MCP608, U5 ESP32-WROOM-32, U6 CY7C65213A-28PVXI

Commit message: left off working on amp
Parts:
- removed G***: LOGO, PCB_ESP32:Garrett_Signature
- removed G***: LOGO, PCB_ESP32:Joe_Signature
- removed G***: LOGO, PCB_ESP32:Molly_Signature
- removed G***: LOGO, PCB_ESP32:Mitch_Signature
- removed G***: LOGO, PCB_ESP32:Logo_inverted
- removed U4: MCP608, Package_DIP:DIP-8_W7.62mm
- added C1: 1uF, Capacitor_SMD:C_0805_2012Metric_Pad1.18x1.45mm_HandSolder, F.Cu at (184.0, 84.2)
- added C2: 0.39uF, Capacitor_SMD:C_0805_2012Metric_Pad1.18x1.45mm_HandSolder, F.Cu at (172.9, 87.9)
- added JP1: Jumper, Connector_PinHeader_2.54mm:PinHeader_1x02_P2.54mm_Vertical, F.Cu at (179.1, 76.9)
- added JP2: Jumper, Connector_PinHeader_2.54mm:PinHeader_1x02_P2.54mm_Vertical, F.Cu at (170.6, 83.6)
- added R1: 20k, Resistor_SMD:R_0805_2012Metric_Pad1.20x1.40mm_HandSolder, F.Cu at (177.6, 79.8)
- added R2: 20k, Resistor_SMD:R_0805_2012Metric_Pad1.20x1.40mm_HandSolder, F.Cu at (177.0, 87.9)
- added R3: 20k, Resistor_SMD:R_0805_2012Metric_Pad1.20x1.40mm_HandSolder, F.Cu at (181.0, 87.9)
- added U2: LM4890, Package_SO:TSSOP-8_3x3mm_P0.65mm, F.Cu at (178.7, 83.9)
- C6: value 10uF -> 1uF; footprint Capacitor_THT:CP_Radial_D5.0mm_P2.50mm -> Capacitor_SMD:C_0805_2012Metric_Pad1.18x1.45mm_HandSolder
- moved C6 10.8 mm to (173.5, 82.5)
- moved H4 2.44 mm to (178.3, 70.1)
Connections:
- C6 pad 1: Net-(C6-Pad1) -> /S_BYPASS
- C6 pad 2: Net-(C6-Pad2) -> GND
- LS1 pad 1: Net-(C6-Pad1) -> Net-(LS1-Pad1)
- LS1 pad 2: GND -> Net-(LS1-Pad2)
- RV1 pad 1: Net-(RV1-Pad1) -> Net-(R3-Pad1)
- RV1 pad 4: Net-(C6-Pad2) -> Net-(R3-Pad1)
- RV1 pad 7: GND -> Net-(LS1-Pad1)
Routing:
- net Net-(RV1-Pad1): track 31.6 -> 0.00 mm, vias 1 -> 0
- net Net-(C6-Pad1): track 30.1 -> 0.00 mm
- net Net-(C6-Pad2): track 15.3 -> 0.00 mm
- net Net-(D2-Pad2): track 45.7 -> 32.8 mm
- net /SPEAKER: track 68.8 -> 61.3 mm
- net /S_BYPASS: track 0.00 -> 6.02 mm
- net Net-(R2-Pad1): track 0.00 -> 2.08 mm
- net Net-(C2-Pad1): track 0.00 -> 2.07 mm
